Commit message: 修改为两个差速轮的模型

File: urdf/diff_drive.urdf (robot description, URDF)
Before this commit: robot diff_drive, 4 links, 3 joints
Links:
- link base_link: geometry collision box size=0.50 0.45 0.12; visual box size=0.50 0.45 0.12
Joints:
- joint caster_joint: origin xyz=-0.18 0 -0.07 rpy=0 0 0 -> xyz=-0.22 0 -0.10 rpy=0 0 0
- joint left_wheel_joint: origin xyz=0 0.18 -0.04 rpy=0 0 0 -> xyz=0 0.25 -0.04 rpy=0 0 0
- joint right_wheel_joint: origin xyz=0 -0.18 -0.04 rpy=0 0 0 -> xyz=0 -0.25 -0.04 rpy=0 0 0

Commit message: 完成step3：加入斜坡地形模型，重建履带车

File: urdf/diff_drive.urdf (robot description, URDF)
Before this commit: robot diff_drive, 4 links, 3 joints
Links:
- link base_link: geometry collision box size=0.68 0.45 0.12; visual box size=0.68 0.45 0.12
Joints:
- joint caster_joint: origin xyz=-0.22 0 -0.10 rpy=0 0 0 -> xyz=0.30 0 -0.10 rpy=0 0 0
- joint left_wheel_joint: origin xyz=0 0.25 -0.04 rpy=0 0 0 -> xyz=-0.12 0.25 -0.04 rpy=0 0 0
- joint right_wheel_joint: origin xyz=0 -0.25 -0.04 rpy=0 0 0 -> xyz=-0.12 -0.25 -0.04 rpy=0 0 0
