Commit message: 阶段4: runSim v2 发布
1. v2正式入口
2. 采集导出
3. 安装验收

File: urdf/active_steering_4wd.urdf (robot description, URDF)
Before this commit: robot active_steering_4wd, 10 links, 9 joints
Links:
- added link lidar_link, mass 0.01; visual cylinder length=0.06 radius=0.055
Joints:
- added joint lidar_link_joint: type fixed, parent base_link, child lidar_link, origin xyz=0 0 0.105

File: urdf/df_back.urdf (robot description, URDF)
Before this commit: robot df_back, 7 links, 6 joints
Links:
- added link lidar_link, mass 0.01; visual cylinder length=0.055 radius=0.055
Joints:
- added joint lidar_link_joint: type fixed, parent base_link, child lidar_link, origin xyz=0 0 0.105

File: urdf/df_front.urdf (robot description, URDF)
Before this commit: robot df_front, 7 links, 6 joints
Links:
- added link lidar_link, mass 0.01; visual cylinder length=0.055 radius=0.055
Joints:
- added joint lidar_link_joint: type fixed, parent base_link, child lidar_link, origin xyz=0 0 0.105

File: urdf/df_mid.urdf (robot description, URDF)
Before this commit: robot df_mid, 8 links, 7 joints
Links:
- added link lidar_link, mass 0.01; visual cylinder length=0.055 radius=0.055
Joints:
- added joint lidar_link_joint: type fixed, parent base_link, child lidar_link, origin xyz=0 0 0.105
- joint front_support_joint: origin xyz=0.30 0 -0.098 -> xyz=0.30 0 -0.096
- joint rear_support_joint: origin xyz=-0.30 0 -0.098 -> xyz=-0.30 0 -0.096
